Commit message: 修改urdf机械臂零点位置

File: src/piper_description/urdf/backup/piper_description copy.urdf (robot description, URDF)
Before this commit: robot piper_description, 9 links, 8 joints
Links:
- link base_link: mass 0.0001 -> None
- link link1: mass 0.0001 -> 0.0978679932242825
- link link2: mass 0.0001 -> 0.289571136953082
- link link3: mass 0.0001 -> 0.290583247455324
- link link4: mass 0.0001 -> 0.127087348341362
- link link5: mass 0.0001 -> 0.144711209371719
- link link6: mass 0.0001 -> 0.150196458571266
- link link7: mass 0.0001 -> 0.0264822500394006
- link link8: mass 0.0001 -> 0.0264822490707451
Joints:
- joint joint1: limit lower=-2.618 upper=2.618 effort=100 velocity=3 -> lower=-2.618 upper=2.618 effort=100 velocity=0
- joint joint2: limit lower=0 upper=3.14 effort=100 velocity=3 -> lower=0 upper=3.14 effort=100 velocity=1
- joint joint3: limit lower=-2.697 upper=0 effort=100 velocity=3 -> lower=-2.967 upper=0 effort=100 velocity=1
- joint joint4: limit lower=-1.832 upper=1.832 effort=100 velocity=3 -> lower=-1.832 upper=1.832 effort=100 velocity=1
- joint joint5: limit lower=-1.22 upper=1.22 effort=100 velocity=3 -> lower=-1.22 upper=1.22 effort=100 velocity=1; origin xyz=0 0 0 rpy=1.5708 0 0 -> xyz=0 0 0 rpy=1.5708 -0.087266 0
- joint joint6: limit lower=-3.14 upper=3.14 effort=100 velocity=3 -> lower=-3.14 upper=3.14 effort=100 velocity=1
- joint joint7: limit lower=0 upper=0.04 effort=10 velocity=1 -> lower=-0.038 upper=0 effort=100 velocity=1
- joint joint8: limit lower=-0.04 upper=0 effort=10 velocity=1 -> lower=0 upper=0.038 effort=100 velocity=1

File: src/piper_description/urdf/backup/piper_description copy.xacro (robot description, xacro)
@@ -1,22 +1,27 @@
 <?xml version="1.0" encoding="utf-8"?>
-<!-- This URDF was automatically created by SolidWorks to URDF Exporter! Originally created by Stephen Brawner (brawner@gmail.com)
-     Commit Version: 1.6.0-4-g7f85cfe  Build Version: 1.6.7995.38578
-     For more information, please see http://wiki.ros.org/sw_urdf_exporter -->
 <robot
-  name="piper_description">
+  name="arm"
+  xmlns:xacro="http://ros.org/wiki/xacro">
+<!-- world -->
+  <link name="world"/>
+  <joint name="fixed_base_joint" type="fixed">
+      <parent link="world"/>
+      <child link="base_link"/>
+  </joint>
+<!-- arm -->
   <link
     name="base_link">
     <inertial>
       <origin
-        xyz="-0.00973928490005031 1.83127089286717E-06 0.0410140167677137"
-        rpy="0 0 0" />
-      <mass
-        value="0.0001" />
+        xyz="-0.00973928490005031 1.8312708928633E-06 0.0410140167677137"
+        rpy="0 0 0" />
+      <mass
+        value="0.00001" />
       <inertia
         ixx="0.000226592553127906"
-        ixy="-7.33974356968615E-08"
-        ixz="2.13221970218122E-06"
+        ixy="-7.33974356968813E-08"
+        ixz="2.13221970218123E-06"
         iyy="0.000269447877479622"
-        iyz="8.15167478682596E-09"
+        iyz="8.15167478685076E-09"
         izz="0.000222318286704" />
     </inertial>
@@ -49,10 +54,10 @@
     <inertial>
       <origin
-        xyz="0.00131676031927021 0.000310288842008365 -0.00922874512303438"
-        rpy="0 0 0" />
-      <mass
-        value="0.0001" />
-      <inertia
-        ixx="7.76684558296782E-05"
+        xyz="0.00131676031927021 0.000310288842008364 -0.00922874512303438"
+        rpy="0 0 0" />
+      <mass
+        value="0.00001" />
+      <inertia
+        ixx="7.76684558296781E-05"
         ixy="1.09084650459916E-07"
         ixz="-1.97480532432411E-06"
@@ -101,5 +106,5 @@
       upper="2.618"
       effort="100"
-      velocity="3" />
+      velocity="1" />
   </joint>
   <link
@@ -107,14 +112,14 @@
     <inertial>
       <origin
-        xyz="0.147615838821413 -0.0174259998251394 0.00175952516190707"
-        rpy="0 0 0" />
-      <mass
-        value="0.0001" />
+        xyz="0.147615838821413 -0.0174259998251393 0.00175952516190707"
+        rpy="0 0 0" />
+      <mass
+        value="0.00001" />
       <inertia
         ixx="0.000150112628108228"
         ixy="8.58974959950769E-05"
-        ixz="-1.07428153464284E-06"
+        ixz="-1.07428153464285E-06"
         iyy="0.00172585302855383"
-        iyz="-9.93704792239676E-07"
+        iyz="-9.93704792239686E-07"
         izz="0.00177445942914759" />
     </inertial>
@@ -159,5 +164,5 @@
       upper="3.14"
       effort="100"
-      velocity="3" />
+      velocity="1" />
   </joint>
   <link
@@ -165,15 +170,15 @@
     <inertial>
       <origin
-        xyz="0.0156727239770991 0.104466514402189 0.000508486576356504"
-        rpy="0 0 0" />
-      <mass
-        value="0.0001" />
-      <inertia
-        ixx="0.00022168634302318"
-        ixy="-7.57426147001315E-06"
-        ixz="-6.36999759250492E-07"
-        iyy="0.000100859159512329"
-        iyz="-8.16199264787698E-07"
-        izz="0.000241839306422341" />
+        xyz="0.0156727246030052 0.104466514905741 0.000508486764144372"
+        rpy="0 0 0" />
+      <mass
+        value="0.00001" />
+      <inertia
+        ixx="0.000221686352136266"
+        ixy="-7.57426543992343E-06"
+        ixz="-6.3700062772173E-07"
+        iyy="0.000100859162015934"
+        iyz="-8.16202696860781E-07"
+        izz="0.000241839316548946" />
     </inertial>
     <visual>
@@ -214,8 +219,8 @@
       xyz="0 0 1" />
     <limit
-      lower="-2.697"
+      lower="-2.967"
       upper="0"
       effort="100"
-      velocity="3" />
+      velocity="1" />
   </joint>
   <link
@@ -223,15 +228,15 @@
     <inertial>
       <origin
-        xyz="0.000276464622388145 -0.00102803669324856 -0.00472830700561582"
-        rpy="0 0 0" />
-      <mass
-        value="0.0001" />
-      <inertia
-        ixx="3.82011730423392E-05"
-        ixy="-4.92358350916331E-08"
-        ixz="4.89589432971791E-08"
-        iyy="4.87048555222583E-05"
-        iyz="6.70802942501353E-08"
-        izz="4.10592077565539E-05" />
+        xyz="0.000276464622388145 -0.00102803669324853 -0.00472830700561612"
+        rpy="0 0 0" />
+      <mass
+        value="0.00001" />
+      <inertia
+        ixx="3.82011730423098E-05"
+        ixy="-4.92358351033589E-08"
+        ixz="4.89589432983109E-08"
+        iyy="4.87048555222491E-05"
+        iyz="6.70802942486707E-08"
+        izz="4.10592077565155E-05" />
     </inertial>
     <visual>
@@ -275,5 +280,5 @@
       upper="1.832"
       effort="100"
-      velocity="3" />
+      velocity="1" />
   </joint>
   <link
@@ -281,15 +286,15 @@
     <inertial>
       <origin
-        xyz="8.82262433637704E-05 0.0566829014808264 -0.00196119720482555"
-        rpy="0 0 0" />
-      <mass
-        value="0.0001" />
-      <inertia
-        ixx="4.39644313661978E-05"
-        ixy="-3.59259686449865E-08"
-        ixz="-1.89747741592145E-08"
-        iyy="5.6317392095077E-05"
-        iyz="-2.1540716689678E-07"
-        izz="4.88713664675246E-05" />
+        xyz="8.82261259100015E-05 0.056682908434204 -0.00196119077436732"
+        rpy="0 0 0" />
+      <mass
+        value="0.00001" />
+      <inertia
+        ixx="4.39644269159173E-05"
+        ixy="-3.59214840853815E-08"
+        ixz="-1.89785003257649E-08"
+        iyy="5.63173857792457E-05"
+        iyz="-2.15407623722543E-07"
+        izz="4.88713595021005E-05" />
     </inertial>
     <visual>
@@ -322,5 +327,5 @@
     <origin
       xyz="0 0 0"
-      rpy="1.5708 0 0" />
+      rpy="1.5708 -0.087266 0" />
     <parent
       link="link4" />
@@ -333,5 +338,5 @@
       upper="1.22"
       effort="100"
-      velocity="3" />
+      velocity="1" />
   </joint>
   <link
@@ -339,15 +344,15 @@
     <inertial>
       <origin
-        xyz="1.16933298222217E-08 0.00034121124902961 0.0342122963963336"
-        rpy="0 0 0" />
-      <mass
-        value="0.0001" />
-      <inertia
-        ixx="4.31750624665837E-05"
-        ixy="-2.21358545270113E-08"
-        ixz="-4.12717194808373E-12"
-        iyy="9.99756712688719E-05"
-        iyz="1.10337149130826E-07"
-        izz="0.000118282337309882" />
+        xyz="9.41121070072333E-09 0.000341209775988838 0.0342122921883722"
+        rpy="0 0 0" />
+      <mass
+        value="0.00001" />
+      <inertia
+        ixx="4.31750564711759E-05"
+        ixy="-2.21295720427027E-08"
+        ixz="-3.27825836857102E-12"
+        iyy="9.99756357365307E-05"
+        iyz="1.10337380549335E-07"
+        izz="0.000118282295533688" />
     </inertial>
     <visual>
@@ -391,5 +396,5 @@
       upper="3.14"
       effort="100"
-      velocity="3" />
+      velocity="1" />
   </joint>
   <link
@@ -397,15 +402,15 @@
     <inertial>
       <origin
-        xyz="-0.00027777838372664 -0.0467673043652057 -0.00921029491873199"
-        rpy="0 0 0" />
-      <mass
-        value="0.0001" />
-      <inertia
-        ixx="9.99787479924596E-06"
-        ixy="-1.57548495096094E-07"
-        ixz="-2.71342775003444E-08"
-        iyy="6.17952122936548E-06"
-        iyz="-1.58939803580081E-06"
-        izz="1.42102717246565E-05" />
+        xyz="-0.000277795893713934 -0.046767350270289 -0.00921029791141448"
+        rpy="0 0 0" />
+      <mass
+        value="0.00001" />
+      <inertia
+        ixx="9.99782519244544E-06"
+        ixy="-1.57547595978589E-07"
+        ixz="-2.71355785017816E-08"
+        iyy="6.17952364356547E-06"
+        iyz="-1.58939504838734E-06"
+        izz="1.42102253390315E-05" />
     </inertial>
     <visual>
@@ -447,6 +452,6 @@
     <limit
       lower="0"
-      upper="0.04"
-      effort="10"
+      upper="0.038"
+      effort="100"
       velocity="1" />
   </joint>
@@ -455,15 +460,15 @@
     <inertial>
       <origin
-        xyz="0.000277816920932594 0.0467673824062785 -0.00921030054507634"
-        rpy="0 0 0" />
-      <mass
-        value="0.0001" />
-      <inertia
-        ixx="9.99779119361565E-06"
-        ixy="-1.5754228345079E-07"
-        ixz="2.7136744671289E-08"
-        iyy="6.17952441558639E-06"
-        iyz="1.58939319453633E-06"
-        izz="1.42101927545622E-05" />
+        xyz="0.000277795911672651 0.0467673513153836 -0.00921029799058583"
+        rpy="0 0 0" />
+      <mass
+        value="0.00001" />
+      <inertia
+        ixx="9.99782474142963E-06"
+        ixy="-1.57547666236405E-07"
+        ixz="2.71355834243046E-08"
+        iyy="6.17952362333486E-06"
+        iyz="1.58939503259658E-06"
+        izz="1.42102248648757E-05" />
     </inertial>
     <visual>
@@ -504,8 +509,63 @@
       xyz="0 0 1" />
     <limit
-      lower="-0.04"
+      lower="-0.038"
       upper="0"
-      effort="10"
-      velocity="1" />
-  </joint>
+      effort="300"
+      velocity="1" />
+  </joint>
+<!-- controller -->
+  <xacro:macro name="transmission_block" params="tran_name joint_name motor_name">
+    <transmission name="${tran_name}">
+        <type>transmission_interface/SimpleTransmission</type>
+        <joint name="${joint_name}">
+            <hardwareInterface>hardware_interface/PositionJointInterface</hardwareInterface>
+        </joint>
+        <actuator name="$motor_name">
+            <hardwareInterface>hardware_interface/PositionJointInterface</hardwareInterface>
+            <mechanicalReduction>1</mechanicalReduction>
+        </actuator>
+    </transmission>
+  </xacro:macro>
+  <xacro:transmission_block tran_name="tran1" joint_name="joint1" motor_name="motor1"/>
+  <xacro:transmission_block tran_name="tran2" joint_name="joint2" motor_name="motor2"/>
+  <xacro:transmission_block tran_name="tran3" joint_name="joint3" motor_name="motor3"/>
+  <xacro:transmission_block tran_name="tran4" joint_name="joint4" motor_name="motor4"/>
+  <xacro:transmission_block tran_name="tran5" joint_name="joint5" motor_name="motor5"/>
+  <xacro:transmission_block tran_name="tran6" joint_name="joint6" motor_name="motor6"/>
+  <xacro:transmission_block tran_name="tran7" joint_name="joint7" motor_name="motor7"/>
+  <xacro:transmission_block tran_name="tran8" joint_name="joint8" motor_name="motor8"/>
+<!-- gazebo -->
+  <gazebo>
+    <plugin name="gazebo_ros_control" filename="libgazebo_ros_control.so">
+        <robotNamespace>/piper_description</robotNamespace>
+        <legacyModeNS>true</legacyModeNS>
+    </plugin>
+  </gazebo>
+  <gazebo reference="base_link">
+    <material>Gazebo/Black</material>
+  </gazebo>
+  <gazebo reference="link1">
+    <material>Gazebo/White</material>
+  </gazebo>
+  <gazebo reference="link2">
+    <material>Gazebo/White</material>
+  </gazebo>
+  <gazebo reference="link3">
+    <material>Gazebo/White</material>
+  </gazebo>
+  <gazebo reference="link4">
+    <material>Gazebo/Black</material>
+  </gazebo>
+  <gazebo reference="link5">
+    <material>Gazebo/White</material>
+  </gazebo>
+  <gazebo reference="link6">
+    <material>Gazebo/White</material>
+  </gazebo>
+  <gazebo reference="link7">
+    <material>Gazebo/Orange</material>
+  </gazebo>
+  <gazebo reference="link8">
+    <material>Gazebo/Orange</material>
+  </gazebo>
 </robot>

File: src/piper_description/urdf/piper_description.xacro (robot description, xacro)
@@ -10,18 +10,18 @@
   </joint>
 <!-- arm -->
-  <link
+<link
     name="base_link">
     <inertial>
       <origin
-        xyz="-0.00973928490005031 1.8312708928633E-06 0.0410140167677137"
-        rpy="0 0 0" />
-      <mass
-        value="0.00001" />
+        xyz="-0.00973928490005031 1.83127089286717E-06 0.0410140167677137"
+        rpy="0 0 0" />
+      <mass
+        value="0.0001" />
       <inertia
         ixx="0.000226592553127906"
-        ixy="-7.33974356968813E-08"
-        ixz="2.13221970218123E-06"
+        ixy="-7.33974356968615E-08"
+        ixz="2.13221970218122E-06"
         iyy="0.000269447877479622"
-        iyz="8.15167478685076E-09"
+        iyz="8.15167478682596E-09"
         izz="0.000222318286704" />
     </inertial>
@@ -54,10 +54,10 @@
     <inertial>
       <origin
-        xyz="0.00131676031927021 0.000310288842008364 -0.00922874512303438"
-        rpy="0 0 0" />
-      <mass
-        value="0.00001" />
-      <inertia
-        ixx="7.76684558296781E-05"
+        xyz="0.00131676031927021 0.000310288842008365 -0.00922874512303438"
+        rpy="0 0 0" />
+      <mass
+        value="0.0001" />
+      <inertia
+        ixx="7.76684558296782E-05"
         ixy="1.09084650459916E-07"
         ixz="-1.97480532432411E-06"
@@ -106,5 +106,5 @@
       upper="2.618"
       effort="100"
-      velocity="1" />
+      velocity="3" />
   </joint>
   <link
@@ -112,14 +112,14 @@
     <inertial>
       <origin
-        xyz="0.147615838821413 -0.0174259998251393 0.00175952516190707"
-        rpy="0 0 0" />
-      <mass
-        value="0.00001" />
+        xyz="0.147615838821413 -0.0174259998251394 0.00175952516190707"
+        rpy="0 0 0" />
+      <mass
+        value="0.0001" />
       <inertia
         ixx="0.000150112628108228"
         ixy="8.58974959950769E-05"
-        ixz="-1.07428153464285E-06"
+        ixz="-1.07428153464284E-06"
         iyy="0.00172585302855383"
-        iyz="-9.93704792239686E-07"
+        iyz="-9.93704792239676E-07"
         izz="0.00177445942914759" />
     </inertial>
@@ -164,5 +164,5 @@
       upper="3.14"
       effort="100"
-      velocity="1" />
+      velocity="3" />
   </joint>
   <link
@@ -170,15 +170,15 @@
     <inertial>
       <origin
-        xyz="0.0156727246030052 0.104466514905741 0.000508486764144372"
-        rpy="0 0 0" />
-      <mass
-        value="0.00001" />
-      <inertia
-        ixx="0.000221686352136266"
-        ixy="-7.57426543992343E-06"
-        ixz="-6.3700062772173E-07"
-        iyy="0.000100859162015934"
-        iyz="-8.16202696860781E-07"
-        izz="0.000241839316548946" />
+        xyz="0.0156727239770991 0.104466514402189 0.000508486576356504"
+        rpy="0 0 0" />
+      <mass
+        value="0.0001" />
+      <inertia
+        ixx="0.00022168634302318"
+        ixy="-7.57426147001315E-06"
+        ixz="-6.36999759250492E-07"
+        iyy="0.000100859159512329"
+        iyz="-8.16199264787698E-07"
+        izz="0.000241839306422341" />
     </inertial>
     <visual>
@@ -219,8 +219,8 @@
       xyz="0 0 1" />
     <limit
-      lower="-2.967"
+      lower="-2.697"
       upper="0"
       effort="100"
-      velocity="1" />
+      velocity="3" />
   </joint>
   <link
@@ -228,15 +228,15 @@
     <inertial>
       <origin
-        xyz="0.000276464622388145 -0.00102803669324853 -0.00472830700561612"
-        rpy="0 0 0" />
-      <mass
-        value="0.00001" />
-      <inertia
-        ixx="3.82011730423098E-05"
-        ixy="-4.92358351033589E-08"
-        ixz="4.89589432983109E-08"
-        iyy="4.87048555222491E-05"
-        iyz="6.70802942486707E-08"
-        izz="4.10592077565155E-05" />
+        xyz="0.000276464622388145 -0.00102803669324856 -0.00472830700561582"
+        rpy="0 0 0" />
+      <mass
+        value="0.0001" />
+      <inertia
+        ixx="3.82011730423392E-05"
+        ixy="-4.92358350916331E-08"
+        ixz="4.89589432971791E-08"
+        iyy="4.87048555222583E-05"
+        iyz="6.70802942501353E-08"
+        izz="4.10592077565539E-05" />
     </inertial>
     <visual>
@@ -275,10 +275,10 @@
       link="link4" />
     <axis
-      xyz="0 0 -1" />
+      xyz="0 0 1" />
     <limit
       lower="-1.832"
       upper="1.832"
       effort="100"
-      velocity="1" />
+      velocity="3" />
   </joint>
   <link
@@ -286,15 +286,15 @@
     <inertial>
       <origin
-        xyz="8.82261259100015E-05 0.056682908434204 -0.00196119077436732"
-        rpy="0 0 0" />
-      <mass
-        value="0.00001" />
-      <inertia
-        ixx="4.39644269159173E-05"
-        ixy="-3.59214840853815E-08"
-        ixz="-1.89785003257649E-08"
-        iyy="5.63173857792457E-05"
-        iyz="-2.15407623722543E-07"
-        izz="4.88713595021005E-05" />
+        xyz="8.82262433637704E-05 0.0566829014808264 -0.00196119720482555"
+        rpy="0 0 0" />
+      <mass
+        value="0.0001" />
+      <inertia
+        ixx="4.39644313661978E-05"
+        ixy="-3.59259686449865E-08"
+        ixz="-1.89747741592145E-08"
+        iyy="5.6317392095077E-05"
+        iyz="-2.1540716689678E-07"
+        izz="4.88713664675246E-05" />
     </inertial>
     <visual>
@@ -327,5 +327,5 @@
     <origin
       xyz="0 0 0"
-      rpy="1.5708 -0.087266 0" />
+      rpy="1.5708 0 0" />
     <parent
       link="link4" />
@@ -338,5 +338,5 @@
       upper="1.22"
       effort="100"
-      velocity="1" />
+      velocity="3" />
   </joint>
   <link
@@ -344,15 +344,15 @@
     <inertial>
       <origin
-        xyz="9.41121070072333E-09 0.000341209775988838 0.0342122921883722"
-        rpy="0 0 0" />
-      <mass
-        value="0.00001" />
-      <inertia
-        ixx="4.31750564711759E-05"
-        ixy="-2.21295720427027E-08"
-        ixz="-3.27825836857102E-12"
-        iyy="9.99756357365307E-05"
-        iyz="1.10337380549335E-07"
-        izz="0.000118282295533688" />
+        xyz="1.16933298222217E-08 0.00034121124902961 0.0342122963963336"
+        rpy="0 0 0" />
+      <mass
+        value="0.0001" />
+      <inertia
+        ixx="4.31750624665837E-05"
+        ixy="-2.21358545270113E-08"
+        ixz="-4.12717194808373E-12"
+        iyy="9.99756712688719E-05"
+        iyz="1.10337149130826E-07"
+        izz="0.000118282337309882" />
     </inertial>
     <visual>
@@ -391,10 +391,10 @@
       link="link6" />
     <axis
-      xyz="0 0 -1" />
+      xyz="0 0 1" />
     <limit
       lower="-3.14"
       upper="3.14"
       effort="100"
-      velocity="1" />
+      velocity="3" />
   </joint>
   <link
@@ -402,15 +402,15 @@
     <inertial>
       <origin
-        xyz="-0.000277795893713934 -0.046767350270289 -0.00921029791141448"
-        rpy="0 0 0" />
-      <mass
-        value="0.00001" />
-      <inertia
-        ixx="9.99782519244544E-06"
-        ixy="-1.57547595978589E-07"
-        ixz="-2.71355785017816E-08"
-        iyy="6.17952364356547E-06"
-        iyz="-1.58939504838734E-06"
-        izz="1.42102253390315E-05" />
+        xyz="-0.00027777838372664 -0.0467673043652057 -0.00921029491873199"
+        rpy="0 0 0" />
+      <mass
+        value="0.0001" />
+      <inertia
+        ixx="9.99787479924596E-06"
+        ixy="-1.57548495096094E-07"
+        ixz="-2.71342775003444E-08"
+        iyy="6.17952122936548E-06"
+        iyz="-1.58939803580081E-06"
+        izz="1.42102717246565E-05" />
     </inertial>
     <visual>
@@ -452,6 +452,6 @@
     <limit
       lower="0"
-      upper="0.038"
-      effort="100"
+      upper="0.04"
+      effort="10"
       velocity="1" />
   </joint>
@@ -460,15 +460,15 @@
     <inertial>
       <origin
-        xyz="0.000277795911672651 0.0467673513153836 -0.00921029799058583"
-        rpy="0 0 0" />
-      <mass
-        value="0.00001" />
-      <inertia
-        ixx="9.99782474142963E-06"
-        ixy="-1.57547666236405E-07"
-        ixz="2.71355834243046E-08"
-        iyy="6.17952362333486E-06"
-        iyz="1.58939503259658E-06"
-        izz="1.42102248648757E-05" />
+        xyz="0.000277816920932594 0.0467673824062785 -0.00921030054507634"
+        rpy="0 0 0" />
+      <mass
+        value="0.0001" />
+      <inertia
+        ixx="9.99779119361565E-06"
+        ixy="-1.5754228345079E-07"
+        ixz="2.7136744671289E-08"
+        iyy="6.17952441558639E-06"
+        iyz="1.58939319453633E-06"
+        izz="1.42101927545622E-05" />
     </inertial>
     <visual>
@@ -509,7 +509,7 @@
       xyz="0 0 1" />
     <limit
-      lower="-0.038"
+      lower="-0.04"
       upper="0"
-      effort="300"
+      effort="10"
       velocity="1" />
   </joint>
