Commit message: 增加没有夹爪的仿真,将夹爪初始位置坐标偏移一点防止碰撞

File: src/piper_description/urdf/moveit/piper_no_gripper_description.urdf (robot description, URDF)
Before this commit: robot piper_description, 9 links, 8 joints
Links:
- removed link link7
- removed link link8
- link link6: geometry collision box size=0.01 0.01 0.01; visual box size=0.01 0.01 0.01
Joints:
- removed joint joint7
- removed joint joint8
- joint joint6: axis 0 0 1 -> (none); limit lower=-3.14 upper=3.14 effort=100 velocity=3 -> (none); type revolute -> fixed

File: src/piper_description/urdf/piper_description.xacro (robot description, xacro)
@@ -442,5 +442,5 @@
     type="prismatic">
     <origin
-      xyz="0 0 0.13503"
+      xyz="-0.0001 0 0.13503"
       rpy="1.5708 0 1.5708" />
     <parent
@@ -500,5 +500,5 @@
     type="prismatic">
     <origin
-      xyz="0 0 0.13503"
+      xyz="0.0001 0 0.13503"
       rpy="-1.5708 0 1.5708" />
     <parent

File: src/piper_description/urdf/piper_no_gripper_description.urdf (robot description, URDF)
Before this commit: robot piper_description, 9 links, 8 joints
Links:
- removed link link6
- removed link link7
- removed link link8
Joints:
- removed joint joint6
- removed joint joint7
- removed joint joint8

File: src/piper_description/urdf/piper_no_gripper_description.xacro (robot description, xacro)
@@ -1,9 +1,14 @@
 <?xml version="1.0" encoding="utf-8"?>
-<!-- This URDF was automatically created by SolidWorks to URDF Exporter! Originally created by Stephen Brawner (brawner@gmail.com)
-     Commit Version: 1.6.0-4-g7f85cfe  Build Version: 1.6.7995.38578
-     For more information, please see http://wiki.ros.org/sw_urdf_exporter -->
 <robot
-  name="piper_description">
-  <link
+  name="arm"
+  xmlns:xacro="http://ros.org/wiki/xacro">
+<!-- world -->
+  <link name="world"/>
+  <joint name="fixed_base_joint" type="fixed">
+      <parent link="world"/>
+      <child link="base_link"/>
+  </joint>
+<!-- arm -->
+<link
     name="base_link">
     <inertial>
@@ -335,177 +340,46 @@
       velocity="3" />
   </joint>
-  <link
-    name="link6">
-    <inertial>
-      <origin
-        xyz="1.16933298222217E-08 0.00034121124902961 0.0342122963963336"
-        rpy="0 0 0" />
-      <mass
-        value="0.0001" />
-      <inertia
-        ixx="4.31750624665837E-05"
-        ixy="-2.21358545270113E-08"
-        ixz="-4.12717194808373E-12"
-        iyy="9.99756712688719E-05"
-        iyz="1.10337149130826E-07"
-        izz="0.000118282337309882" />
-    </inertial>
-    <visual>
-      <origin
-        xyz="0 0 0"
-        rpy="0 0 0" />
-      <geometry>
-        <mesh
-          filename="package://piper_description/meshes/link6.STL" />
-      </geometry>
-      <material
-        name="">
-        <color
-          rgba="0.792156862745098 0.819607843137255 0.933333333333333 1" />
-      </material>
-    </visual>
-    <collision>
-      <origin
-        xyz="0 0 0"
-        rpy="0 0 0" />
-      <geometry>
-        <mesh
-          filename="package://piper_description/meshes/link6.STL" />
-      </geometry>
-    </collision>
-  </link>
-  <joint
-    name="joint6"
-    type="revolute">
-    <origin
-      xyz="0 0.091 0.0014165"
-      rpy="-1.5708 -1.5708 0" />
-    <parent
-      link="link5" />
-    <child
-      link="link6" />
-    <axis
-      xyz="0 0 1" />
-    <limit
-      lower="-3.14"
-      upper="3.14"
-      effort="100"
-      velocity="3" />
-  </joint>
-  <link
-    name="link7">
-    <inertial>
-      <origin
-        xyz="-0.00027777838372664 -0.0467673043652057 -0.00921029491873199"
-        rpy="0 0 0" />
-      <mass
-        value="0.0001" />
-      <inertia
-        ixx="9.99787479924596E-06"
-        ixy="-1.57548495096094E-07"
-        ixz="-2.71342775003444E-08"
-        iyy="6.17952122936548E-06"
-        iyz="-1.58939803580081E-06"
-        izz="1.42102717246565E-05" />
-    </inertial>
-    <visual>
-      <origin
-        xyz="0 0 0"
-        rpy="0 0 0" />
-      <geometry>
-        <mesh
-          filename="package://piper_description/meshes/link7.STL" />
-      </geometry>
-      <material
-        name="">
-        <color
-          rgba="0.792156862745098 0.819607843137255 0.933333333333333 1" />
-      </material>
-    </visual>
-    <collision>
-      <origin
-        xyz="0 0 0"
-        rpy="0 0 0" />
-      <geometry>
-        <mesh
-          filename="package://piper_description/meshes/link7.STL" />
-      </geometry>
-    </collision>
-  </link>
-  <joint
-    name="joint7"
-    type="prismatic">
-    <origin
-      xyz="-0.0001 0 0.13503"
-      rpy="1.5708 0 1.5708" />
-    <parent
-      link="link6" />
-    <child
-      link="link7" />
-    <axis
-      xyz="0 0 -1" />
-    <limit
-      lower="0"
-      upper="0.04"
-      effort="10"
-      velocity="1" />
-  </joint>
-  <link
-    name="link8">
-    <inertial>
-      <origin
-        xyz="0.000277816920932594 0.0467673824062785 -0.00921030054507634"
-        rpy="0 0 0" />
-      <mass
-        value="0.0001" />
-      <inertia
-        ixx="9.99779119361565E-06"
-        ixy="-1.5754228345079E-07"
-        ixz="2.7136744671289E-08"
-        iyy="6.17952441558639E-06"
-        iyz="1.58939319453633E-06"
-        izz="1.42101927545622E-05" />
-    </inertial>
-    <visual>
-      <origin
-        xyz="0 0 0"
-        rpy="0 0 0" />
-      <geometry>
-        <mesh
-          filename="package://piper_description/meshes/link8.STL" />
-      </geometry>
-      <material
-        name="">
-        <color
-          rgba="0.792156862745098 0.819607843137255 0.933333333333333 1" />
-      </material>
-    </visual>
-    <collision>
-      <origin
-        xyz="0 0 0"
-        rpy="0 0 0" />
-      <geometry>
-        <mesh
-          filename="package://piper_description/meshes/link8.STL" />
-      </geometry>
-    </collision>
-  </link>
-  <joint
-    name="joint8"
-    type="prismatic">
-    <origin
-      xyz="0.0001 0 0.13503"
-      rpy="-1.5708 0 1.5708" />
-    <parent
-      link="link6" />
-    <child
-      link="link8" />
-    <axis
-      xyz="0 0 1" />
-    <limit
-      lower="-0.04"
-      upper="0"
-      effort="10"
-      velocity="1" />
-  </joint>
+<!-- controller -->
+  <xacro:macro name="transmission_block" params="tran_name joint_name motor_name">
+    <transmission name="${tran_name}">
+        <type>transmission_interface/SimpleTransmission</type>
+        <joint name="${joint_name}">
+            <hardwareInterface>hardware_interface/PositionJointInterface</hardwareInterface>
+        </joint>
+        <actuator name="$motor_name">
+            <hardwareInterface>hardware_interface/PositionJointInterface</hardwareInterface>
+            <mechanicalReduction>1</mechanicalReduction>
+        </actuator>
+    </transmission>
+  </xacro:macro>
+  <xacro:transmission_block tran_name="tran1" joint_name="joint1" motor_name="motor1"/>
+  <xacro:transmission_block tran_name="tran2" joint_name="joint2" motor_name="motor2"/>
+  <xacro:transmission_block tran_name="tran3" joint_name="joint3" motor_name="motor3"/>
+  <xacro:transmission_block tran_name="tran4" joint_name="joint4" motor_name="motor4"/>
+  <xacro:transmission_block tran_name="tran5" joint_name="joint5" motor_name="motor5"/>
+<!-- gazebo -->
+  <gazebo>
+    <plugin name="gazebo_ros_control" filename="libgazebo_ros_control.so">
+        <robotNamespace>/piper_description</robotNamespace>
+        <legacyModeNS>true</legacyModeNS>
+    </plugin>
+  </gazebo>
+  <gazebo reference="base_link">
+    <material>Gazebo/Black</material>
+  </gazebo>
+  <gazebo reference="link1">
+    <material>Gazebo/White</material>
+  </gazebo>
+  <gazebo reference="link2">
+    <material>Gazebo/White</material>
+  </gazebo>
+  <gazebo reference="link3">
+    <material>Gazebo/White</material>
+  </gazebo>
+  <gazebo reference="link4">
+    <material>Gazebo/Black</material>
+  </gazebo>
+  <gazebo reference="link5">
+    <material>Gazebo/White</material>
+  </gazebo>
 </robot>
