Commit message: 修改URDF零点和实际机械臂零点不同的问题

File: src/piper_description/urdf/piper_no_gripper_description_v00.xacro (robot description, xacro)
@@ -1,10 +1,14 @@
 <?xml version="1.0" encoding="utf-8"?>
-<!-- This URDF was automatically created by SolidWorks to URDF Exporter! Originally created by Stephen Brawner (brawner@gmail.com)
-     Commit Version: 1.6.0-4-g7f85cfe  Build Version: 1.6.7995.38578
-     For more information, please see http://wiki.ros.org/sw_urdf_exporter -->
 <robot
-  name="piper_description">
-  <link name="dummy_root" />
-  <link
+  name="arm"
+  xmlns:xacro="http://ros.org/wiki/xacro">
+<!-- world -->
+  <link name="world"/>
+  <joint name="fixed_base_joint" type="fixed">
+      <parent link="world"/>
+      <child link="base_link"/>
+  </joint>
+<!-- arm -->
+<link
     name="base_link">
     <inertial>
@@ -25,4 +29,18 @@
       <origin
         xyz="0 0 0"
+        rpy="1.5708 0 -1.5708" />
+      <geometry>
+        <mesh
+          filename="package://piper_description/meshes/base_link.dae" />
+      </geometry>
+      <material
+        name="">
+        <color
+          rgba="0.792156862745098 0.819607843137255 0.933333333333333 1" />
+      </material>
+    </visual>
+    <collision>
+      <origin
+        xyz="0 0 0"
         rpy="0 0 0" />
       <geometry>
@@ -30,25 +48,6 @@
           filename="package://piper_description/meshes/base_link.STL" />
       </geometry>
-      <material
-        name="">
-        <color
-          rgba="0.792156862745098 0.819607843137255 0.933333333333333 1" />
-      </material>
-    </visual>
-    <collision>
-      <origin
-        xyz="0 0 0"
-        rpy="0 0 0" />
-      <geometry>
-        <mesh
-          filename="package://piper_description/meshes/base_link.STL" />
-      </geometry>
-    </collision>
-  </link>
-    <joint name="fixed_base" type="fixed">
-    <parent link="dummy_root" />
-    <child link="base_link" />
-    <origin xyz="0 0 0" rpy="0 0 0" />
-  </joint>
+    </collision>
+  </link>
   <link
     name="link1">
@@ -70,8 +69,8 @@
       <origin
         xyz="0 0 0"
-        rpy="0 0 0" />
-      <geometry>
-        <mesh
-          filename="package://piper_description/meshes/link1.STL" />
+        rpy="1.5708 0 0" />
+      <geometry>
+        <mesh
+          filename="package://piper_description/meshes/link1.dae" />
       </geometry>
       <material
@@ -128,4 +127,18 @@
       <origin
         xyz="0 0 0"
+        rpy="0 1.5708 -0.0873" />
+      <geometry>
+        <mesh
+          filename="package://piper_description/meshes/link2.dae" />
+      </geometry>
+      <material
+        name="">
+        <color
+          rgba="0.792156862745098 0.819607843137255 0.933333333333333 1" />
+      </material>
+    </visual>
+    <collision>
+      <origin
+        xyz="0 0 0"
         rpy="0 0 0" />
       <geometry>
@@ -133,18 +146,4 @@
           filename="package://piper_description/meshes/link2.STL" />
       </geometry>
-      <material
-        name="">
-        <color
-          rgba="0.792156862745098 0.819607843137255 0.933333333333333 1" />
-      </material>
-    </visual>
-    <collision>
-      <origin
-        xyz="0 0 0"
-        rpy="0 0 0" />
-      <geometry>
-        <mesh
-          filename="package://piper_description/meshes/link2.STL" />
-      </geometry>
     </collision>
   </link>
@@ -152,7 +151,10 @@
     name="joint2"
     type="revolute">
-    <origin
+    <!-- <origin
       xyz="0 0 0"
-      rpy="1.5708 -0.10095 -1.5708" />
+      rpy="1.5708 -0.10095 -1.5708" /> -->
+    <origin
+      xyz="0 0 0"
+      rpy="1.5708 -0.135857 -1.5708" />
     <parent
       link="link1" />
@@ -186,4 +188,18 @@
       <origin
         xyz="0 0 0"
+        rpy="1.4835 1.5708 0" />
+      <geometry>
+        <mesh
+          filename="package://piper_description/meshes/link3.dae" />
+      </geometry>
+      <material
+        name="">
+        <color
+          rgba="0.792156862745098 0.819607843137255 0.933333333333333 1" />
+      </material>
+    </visual>
+    <collision>
+      <origin
+        xyz="0 0 0"
         rpy="0 0 0" />
       <geometry>
@@ -191,18 +207,4 @@
           filename="package://piper_description/meshes/link3.STL" />
       </geometry>
-      <material
-        name="">
-        <color
-          rgba="0.792156862745098 0.819607843137255 0.933333333333333 1" />
-      </material>
-    </visual>
-    <collision>
-      <origin
-        xyz="0 0 0"
-        rpy="0 0 0" />
-      <geometry>
-        <mesh
-          filename="package://piper_description/meshes/link3.STL" />
-      </geometry>
     </collision>
   </link>
@@ -210,7 +212,10 @@
     name="joint3"
     type="revolute">
-    <origin
+    <!-- <origin
       xyz="0.28503 0 0"
-      rpy="0 0 1.3826" />
+      rpy="0 0 1.3826" /> -->
+    <origin
+      xyz="0.28503 0 0"
+      rpy="0 0 1.347693" />
     <parent
       link="link2" />
@@ -244,8 +249,8 @@
       <origin
         xyz="0 0 0"
-        rpy="0 0 0" />
-      <geometry>
-        <mesh
-          filename="package://piper_description/meshes/link4.STL" />
+        rpy="1.48 0 1.5708" />
+      <geometry>
+        <mesh
+          filename="package://piper_description/meshes/link4.dae" />
       </geometry>
       <material
@@ -302,8 +307,8 @@
       <origin
         xyz="0 0 0"
-        rpy="0 0 0" />
-      <geometry>
-        <mesh
-          filename="package://piper_description/meshes/link5.STL" />
+        rpy="1.4835 1.5708 0" />
+      <geometry>
+        <mesh
+          filename="package://piper_description/meshes/link5.dae" />
       </geometry>
       <material
@@ -341,30 +346,46 @@
       velocity="3" />
   </joint>
-  <link name="link6">
-    <inertial>
-      <origin xyz="0 0 0" rpy="0 0 0" />
-      <mass value="0.0001" />
-      <inertia ixx="1e-6" ixy="0" ixz="0" iyy="1e-6" iyz="0" izz="1e-6" />
-    </inertial>
-    <visual>
-      <origin xyz="0 0 -0.01" rpy="0 0 0" />
-      <geometry>
-        <box size="0.01 0.01 0.01" />  <!-- 小方块尺寸 -->
-      </geometry>
-      <material name="">
-        <color rgba="0.792 0.819 0.933 1" />
-      </material>
-    </visual>
-    <collision>
-      <origin xyz="0 0 0" rpy="0 0 0" />
-      <geometry>
-        <box size="0.01 0.01 0.01" />  <!-- 小方块尺寸 -->
-      </geometry>
-    </collision>
-  </link>
-  <joint name="joint6" type="fixed">
-    <origin xyz="0 0.091 0.0014165" rpy="-1.5708 -1.5708 0" />
-    <parent link="link5" />
-    <child link="link6" />
-  </joint>
+<!-- controller -->
+  <xacro:macro name="transmission_block" params="tran_name joint_name motor_name">
+    <transmission name="${tran_name}">
+        <type>transmission_interface/SimpleTransmission</type>
+        <joint name="${joint_name}">
+            <hardwareInterface>hardware_interface/PositionJointInterface</hardwareInterface>
+        </joint>
+        <actuator name="$motor_name">
+            <hardwareInterface>hardware_interface/PositionJointInterface</hardwareInterface>
+            <mechanicalReduction>1</mechanicalReduction>
+        </actuator>
+    </transmission>
+  </xacro:macro>
+  <xacro:transmission_block tran_name="tran1" joint_name="joint1" motor_name="motor1"/>
+  <xacro:transmission_block tran_name="tran2" joint_name="joint2" motor_name="motor2"/>
+  <xacro:transmission_block tran_name="tran3" joint_name="joint3" motor_name="motor3"/>
+  <xacro:transmission_block tran_name="tran4" joint_name="joint4" motor_name="motor4"/>
+  <xacro:transmission_block tran_name="tran5" joint_name="joint5" motor_name="motor5"/>
+<!-- gazebo -->
+  <gazebo>
+    <plugin name="gazebo_ros_control" filename="libgazebo_ros_control.so">
+        <robotNamespace>/piper_description</robotNamespace>
+        <legacyModeNS>true</legacyModeNS>
+    </plugin>
+  </gazebo>
+  <gazebo reference="base_link">
+    <material>Gazebo/Black</material>
+  </gazebo>
+  <gazebo reference="link1">
+    <material>Gazebo/White</material>
+  </gazebo>
+  <gazebo reference="link2">
+    <material>Gazebo/White</material>
+  </gazebo>
+  <gazebo reference="link3">
+    <material>Gazebo/White</material>
+  </gazebo>
+  <gazebo reference="link4">
+    <material>Gazebo/Black</material>
+  </gazebo>
+  <gazebo reference="link5">
+    <material>Gazebo/White</material>
+  </gazebo>
 </robot>
