Commit message: 增加urdf的dae

File: src/piper_description/urdf/piper_description.urdf (robot description, URDF)
Before this commit: robot piper_description, 9 links, 8 joints
Links:
- link base_link: geometry collision mesh filename=package://piper_description/meshes/base_link.STL; visual mesh filename=package://piper_description/meshes/base_link.dae
- link link1: geometry collision mesh filename=package://piper_description/meshes/link1.STL; visual mesh filename=package://piper_description/meshes/link1.dae
- link link2: geometry collision mesh filename=package://piper_description/meshes/link2.STL; visual mesh filename=package://piper_description/meshes/link2.dae
- link link3: geometry collision mesh filename=package://piper_description/meshes/link3.STL; visual mesh filename=package://piper_description/meshes/link3.dae
- link link4: geometry collision mesh filename=package://piper_description/meshes/link4.STL; visual mesh filename=package://piper_description/meshes/link4.dae
- link link5: geometry collision mesh filename=package://piper_description/meshes/link5.STL; visual mesh filename=package://piper_description/meshes/link5.dae
- link link6: geometry collision mesh filename=package://piper_description/meshes/link6.STL; visual mesh filename=package://piper_description/meshes/link6.dae
- link link7: geometry collision mesh filename=package://piper_description/meshes/link7.STL; visual mesh filename=package://piper_description/meshes/link7.dae
- link link8: geometry collision mesh filename=package://piper_description/meshes/link8.STL; visual mesh filename=package://piper_description/meshes/link8.dae

File: src/piper_description/urdf/piper_description.xacro (robot description, xacro)
@@ -29,8 +29,8 @@
       <origin
         xyz="0 0 0"
-        rpy="0 0 0" />
-      <geometry>
-        <mesh
-          filename="package://piper_description/meshes/base_link.STL" />
+        rpy="1.5708 0 -1.5708" />
+      <geometry>
+        <mesh
+          filename="package://piper_description/meshes/base_link.dae" />
       </geometry>
       <material
@@ -69,8 +69,8 @@
       <origin
         xyz="0 0 0"
-        rpy="0 0 0" />
-      <geometry>
-        <mesh
-          filename="package://piper_description/meshes/link1.STL" />
+        rpy="1.5708 0 0" />
+      <geometry>
+        <mesh
+          filename="package://piper_description/meshes/link1.dae" />
       </geometry>
       <material
@@ -127,8 +127,8 @@
       <origin
         xyz="0 0 0"
-        rpy="0 0 0" />
-      <geometry>
-        <mesh
-          filename="package://piper_description/meshes/link2.STL" />
+        rpy="0 1.5708 -0.0873" />
+      <geometry>
+        <mesh
+          filename="package://piper_description/meshes/link2.dae" />
       </geometry>
       <material
@@ -185,8 +185,8 @@
       <origin
         xyz="0 0 0"
-        rpy="0 0 0" />
-      <geometry>
-        <mesh
-          filename="package://piper_description/meshes/link3.STL" />
+        rpy="1.4835 1.5708 0" />
+      <geometry>
+        <mesh
+          filename="package://piper_description/meshes/link3.dae" />
       </geometry>
       <material
@@ -243,8 +243,8 @@
       <origin
         xyz="0 0 0"
-        rpy="0 0 0" />
-      <geometry>
-        <mesh
-          filename="package://piper_description/meshes/link4.STL" />
+        rpy="1.48 0 1.5708" />
+      <geometry>
+        <mesh
+          filename="package://piper_description/meshes/link4.dae" />
       </geometry>
       <material
@@ -301,8 +301,8 @@
       <origin
         xyz="0 0 0"
-        rpy="0 0 0" />
-      <geometry>
-        <mesh
-          filename="package://piper_description/meshes/link5.STL" />
+        rpy="1.5 1.5708 0" />
+      <geometry>
+        <mesh
+          filename="package://piper_description/meshes/link5.dae" />
       </geometry>
       <material
@@ -359,8 +359,8 @@
       <origin
         xyz="0 0 0"
-        rpy="0 0 0" />
-      <geometry>
-        <mesh
-          filename="package://piper_description/meshes/link6.STL" />
+        rpy="3.14159 0 3.14159" />
+      <geometry>
+        <mesh
+          filename="package://piper_description/meshes/link6.dae" />
       </geometry>
       <material
@@ -417,8 +417,8 @@
       <origin
         xyz="0 0 0"
-        rpy="0 0 0" />
-      <geometry>
-        <mesh
-          filename="package://piper_description/meshes/link7.STL" />
+        rpy="-0.0873 -1.5708 1.5708" />
+      <geometry>
+        <mesh
+          filename="package://piper_description/meshes/link7.dae" />
       </geometry>
       <material
@@ -475,8 +475,8 @@
       <origin
         xyz="0 0 0"
-        rpy="0 0 0" />
-      <geometry>
-        <mesh
-          filename="package://piper_description/meshes/link8.STL" />
+        rpy="-0.0873 1.5708 1.5708" />
+      <geometry>
+        <mesh
+          filename="package://piper_description/meshes/link8.dae" />
       </geometry>
       <material

File: src/piper_description/urdf/piper_no_gripper_description.urdf (robot description, URDF)
Before this commit: robot piper_description, 6 links, 5 joints
Links:
- link base_link: geometry collision mesh filename=package://piper_description/meshes/base_link.STL; visual mesh filename=package://piper_description/meshes/base_link.dae
- link link1: geometry collision mesh filename=package://piper_description/meshes/link1.STL; visual mesh filename=package://piper_description/meshes/link1.dae
- link link2: geometry collision mesh filename=package://piper_description/meshes/link2.STL; visual mesh filename=package://piper_description/meshes/link2.dae
- link link3: geometry collision mesh filename=package://piper_description/meshes/link3.STL; visual mesh filename=package://piper_description/meshes/link3.dae
- link link4: geometry collision mesh filename=package://piper_description/meshes/link4.STL; visual mesh filename=package://piper_description/meshes/link4.dae
- link link5: geometry collision mesh filename=package://piper_description/meshes/link5.STL; visual mesh filename=package://piper_description/meshes/link5.dae

File: src/piper_description/urdf/piper_no_gripper_description.xacro (robot description, xacro)
@@ -29,8 +29,8 @@
       <origin
         xyz="0 0 0"
-        rpy="0 0 0" />
-      <geometry>
-        <mesh
-          filename="package://piper_description/meshes/base_link.STL" />
+        rpy="1.5708 0 -1.5708" />
+      <geometry>
+        <mesh
+          filename="package://piper_description/meshes/base_link.dae" />
       </geometry>
       <material
@@ -69,8 +69,8 @@
       <origin
         xyz="0 0 0"
-        rpy="0 0 0" />
-      <geometry>
-        <mesh
-          filename="package://piper_description/meshes/link1.STL" />
+        rpy="1.5708 0 0" />
+      <geometry>
+        <mesh
+          filename="package://piper_description/meshes/link1.dae" />
       </geometry>
       <material
@@ -127,8 +127,8 @@
       <origin
         xyz="0 0 0"
-        rpy="0 0 0" />
-      <geometry>
-        <mesh
-          filename="package://piper_description/meshes/link2.STL" />
+        rpy="0 1.5708 -0.0873" />
+      <geometry>
+        <mesh
+          filename="package://piper_description/meshes/link2.dae" />
       </geometry>
       <material
@@ -185,8 +185,8 @@
       <origin
         xyz="0 0 0"
-        rpy="0 0 0" />
-      <geometry>
-        <mesh
-          filename="package://piper_description/meshes/link3.STL" />
+        rpy="1.4835 1.5708 0" />
+      <geometry>
+        <mesh
+          filename="package://piper_description/meshes/link3.dae" />
       </geometry>
       <material
@@ -243,8 +243,8 @@
       <origin
         xyz="0 0 0"
-        rpy="0 0 0" />
-      <geometry>
-        <mesh
-          filename="package://piper_description/meshes/link4.STL" />
+        rpy="1.48 0 1.5708" />
+      <geometry>
+        <mesh
+          filename="package://piper_description/meshes/link4.dae" />
       </geometry>
       <material
@@ -301,8 +301,8 @@
       <origin
         xyz="0 0 0"
-        rpy="0 0 0" />
-      <geometry>
-        <mesh
-          filename="package://piper_description/meshes/link5.STL" />
+        rpy="1.5 1.5708 0" />
+      <geometry>
+        <mesh
+          filename="package://piper_description/meshes/link5.dae" />
       </geometry>
       <material

Commit message: 将dae颜色变浅,修改readme

File: src/piper_description/urdf/piper_description.urdf (robot description, URDF)
Before this commit: robot piper_description, 9 links, 8 joints
Links:
- link base_link: mass 0.0001 -> 0.162352169522719
- link link1: mass 0.0001 -> 0.0978679932242825
- link link2: mass 0.0001 -> 0.289571136953082
- link link3: mass 0.0001 -> 0.290583243387798
- link link4: mass 0.0001 -> 0.127087348341362
- link link5: mass 0.0001 -> 0.144711242639456
- link link6: mass 0.0001 -> 0.150196493124859
- link link7: mass 0.0001 -> 0.0264822923452701
- link link8: mass 0.0001 -> 0.0264822021416581
Joints:
- joint joint6: axis 0 0 1 -> 0 0 -1

File: src/piper_description/urdf/piper_description.xacro (robot description, xacro)
@@ -17,5 +17,5 @@
         rpy="0 0 0" />
       <mass
-        value="0.0001" />
+        value="0.162352169522719" />
       <inertia
         ixx="0.000226592553127906"
@@ -29,5 +29,5 @@
       <origin
         xyz="0 0 0"
-        rpy="1.5708 0 -1.5708" />
+        rpy="0 0 0" />
       <geometry>
         <mesh
@@ -57,5 +57,5 @@
         rpy="0 0 0" />
       <mass
-        value="0.0001" />
+        value="0.0978679932242825" />
       <inertia
         ixx="7.76684558296782E-05"
@@ -69,5 +69,5 @@
       <origin
         xyz="0 0 0"
-        rpy="1.5708 0 0" />
+        rpy="0 0 0" />
       <geometry>
         <mesh
@@ -115,5 +115,5 @@
         rpy="0 0 0" />
       <mass
-        value="0.0001" />
+        value="0.289571136953082" />
       <inertia
         ixx="0.000150112628108228"
@@ -127,5 +127,5 @@
       <origin
         xyz="0 0 0"
-        rpy="0 1.5708 -0.0873" />
+        rpy="0 0 0" />
       <geometry>
         <mesh
@@ -173,5 +173,5 @@
         rpy="0 0 0" />
       <mass
-        value="0.0001" />
+        value="0.290583243387798" />
       <inertia
         ixx="0.00022168634302318"
@@ -185,5 +185,5 @@
       <origin
         xyz="0 0 0"
-        rpy="1.4835 1.5708 0" />
+        rpy="0 0 0" />
       <geometry>
         <mesh
@@ -231,5 +231,5 @@
         rpy="0 0 0" />
       <mass
-        value="0.0001" />
+        value="0.127087348341362" />
       <inertia
         ixx="3.82011730423392E-05"
@@ -243,5 +243,5 @@
       <origin
         xyz="0 0 0"
-        rpy="1.48 0 1.5708" />
+        rpy="0 0 0" />
       <geometry>
         <mesh
@@ -289,5 +289,5 @@
         rpy="0 0 0" />
       <mass
-        value="0.0001" />
+        value="0.144711242639456" />
       <inertia
         ixx="4.39644313661978E-05"
@@ -301,5 +301,5 @@
       <origin
         xyz="0 0 0"
-        rpy="1.4835 1.5708 0" />
+        rpy="0 0 0" />
       <geometry>
         <mesh
@@ -347,5 +347,5 @@
         rpy="0 0 0" />
       <mass
-        value="0.0001" />
+        value="0.150196493124859" />
       <inertia
         ixx="4.31750624665837E-05"
@@ -359,5 +359,5 @@
       <origin
         xyz="0 0 0"
-        rpy="3.14159 0 3.14159" />
+        rpy="0 0 0" />
       <geometry>
         <mesh
@@ -391,5 +391,5 @@
       link="link6" />
     <axis
-      xyz="0 0 1" />
+      xyz="0 0 -1" />
     <limit
       lower="-3.14"
@@ -405,5 +405,5 @@
         rpy="0 0 0" />
       <mass
-        value="0.0001" />
+        value="0.0264822923452701" />
       <inertia
         ixx="9.99787479924596E-06"
@@ -417,5 +417,5 @@
       <origin
         xyz="0 0 0"
-        rpy="-0.0873 -1.5708 1.5708" />
+        rpy="0 0 0" />
       <geometry>
         <mesh
@@ -463,5 +463,5 @@
         rpy="0 0 0" />
       <mass
-        value="0.0001" />
+        value="0.0264822021416581" />
       <inertia
         ixx="9.99779119361565E-06"
@@ -475,5 +475,5 @@
       <origin
         xyz="0 0 0"
-        rpy="-0.0873 1.5708 1.5708" />
+        rpy="0 0 0" />
       <geometry>
         <mesh
@@ -542,5 +542,5 @@
     </plugin>
   </gazebo>
-  <gazebo reference="base_link">
+  <!-- <gazebo reference="base_link">
     <material>Gazebo/Black</material>
   </gazebo>
@@ -568,4 +568,4 @@
   <gazebo reference="link8">
     <material>Gazebo/Orange</material>
-  </gazebo>
+  </gazebo> -->
 </robot>

File: src/piper_description/urdf/piper_description_v00.urdf (robot description, URDF)
Before this commit: robot piper_description, 9 links, 8 joints
Links:
- link base_link: mass 0.0001 -> 0.162352169522719
- link link1: mass 0.0001 -> 0.0978679932242825
- link link2: mass 0.0001 -> 0.289571136953082
- link link3: mass 0.0001 -> 0.290583243387798
- link link4: mass 0.0001 -> 0.127087348341362
- link link5: mass 0.0001 -> 0.144711242639456
- link link6: mass 0.0001 -> 0.150196493124859
- link link7: mass 0.0001 -> 0.0264822923452701
- link link8: mass 0.0001 -> 0.0264822021416581
Joints:
- joint joint6: axis 0 0 1 -> 0 0 -1

File: src/piper_description/urdf/piper_description_v00.xacro (robot description, xacro)
@@ -17,5 +17,5 @@
         rpy="0 0 0" />
       <mass
-        value="0.0001" />
+        value="0.162352169522719" />
       <inertia
         ixx="0.000226592553127906"
@@ -29,5 +29,5 @@
       <origin
         xyz="0 0 0"
-        rpy="1.5708 0 -1.5708" />
+        rpy="0 0 0" />
       <geometry>
         <mesh
@@ -57,5 +57,5 @@
         rpy="0 0 0" />
       <mass
-        value="0.0001" />
+        value="0.0978679932242825" />
       <inertia
         ixx="7.76684558296782E-05"
@@ -69,5 +69,5 @@
       <origin
         xyz="0 0 0"
-        rpy="1.5708 0 0" />
+        rpy="0 0 0" />
       <geometry>
         <mesh
@@ -115,5 +115,5 @@
         rpy="0 0 0" />
       <mass
-        value="0.0001" />
+        value="0.289571136953082" />
       <inertia
         ixx="0.000150112628108228"
@@ -127,5 +127,5 @@
       <origin
         xyz="0 0 0"
-        rpy="0 1.5708 -0.0873" />
+        rpy="0 0 0" />
       <geometry>
         <mesh
@@ -176,5 +176,5 @@
         rpy="0 0 0" />
       <mass
-        value="0.0001" />
+        value="0.290583243387798" />
       <inertia
         ixx="0.00022168634302318"
@@ -188,5 +188,5 @@
       <origin
         xyz="0 0 0"
-        rpy="1.4835 1.5708 0" />
+        rpy="0 0 0" />
       <geometry>
         <mesh
@@ -237,5 +237,5 @@
         rpy="0 0 0" />
       <mass
-        value="0.0001" />
+        value="0.127087348341362" />
       <inertia
         ixx="3.82011730423392E-05"
@@ -249,5 +249,5 @@
       <origin
         xyz="0 0 0"
-        rpy="1.48 0 1.5708" />
+        rpy="0 0 0" />
       <geometry>
         <mesh
@@ -295,5 +295,5 @@
         rpy="0 0 0" />
       <mass
-        value="0.0001" />
+        value="0.144711242639456" />
       <inertia
         ixx="4.39644313661978E-05"
@@ -307,5 +307,5 @@
       <origin
         xyz="0 0 0"
-        rpy="1.4835 1.5708 0" />
+        rpy="0 0 0" />
       <geometry>
         <mesh
@@ -353,5 +353,5 @@
         rpy="0 0 0" />
       <mass
-        value="0.0001" />
+        value="0.150196493124859" />
       <inertia
         ixx="4.31750624665837E-05"
@@ -365,5 +365,5 @@
       <origin
         xyz="0 0 0"
-        rpy="3.14159 0 3.14159" />
+        rpy="0 0 0" />
       <geometry>
         <mesh
@@ -397,5 +397,5 @@
       link="link6" />
     <axis
-      xyz="0 0 1" />
+      xyz="0 0 -1" />
     <limit
       lower="-3.14"
@@ -411,5 +411,5 @@
         rpy="0 0 0" />
       <mass
-        value="0.0001" />
+        value="0.0264822923452701" />
       <inertia
         ixx="9.99787479924596E-06"
@@ -423,5 +423,5 @@
       <origin
         xyz="0 0 0"
-        rpy="-0.0873 -1.5708 1.5708" />
+        rpy="0 0 0" />
       <geometry>
         <mesh
@@ -469,5 +469,5 @@
         rpy="0 0 0" />
       <mass
-        value="0.0001" />
+        value="0.0264822021416581" />
       <inertia
         ixx="9.99779119361565E-06"
@@ -481,5 +481,5 @@
       <origin
         xyz="0 0 0"
-        rpy="-0.0873 1.5708 1.5708" />
+        rpy="0 0 0" />
       <geometry>
         <mesh
@@ -548,5 +548,5 @@
     </plugin>
   </gazebo>
-  <gazebo reference="base_link">
+  <!-- <gazebo reference="base_link">
     <material>Gazebo/Black</material>
   </gazebo>
@@ -574,4 +574,4 @@
   <gazebo reference="link8">
     <material>Gazebo/Orange</material>
-  </gazebo>
+  </gazebo> -->
 </robot>

File: src/piper_description/urdf/piper_no_gripper_description.urdf (robot description, URDF)
Before this commit: robot piper_description, 6 links, 5 joints
Links:
- link base_link: mass 0.0001 -> 0.162352169522719
- link link1: mass 0.0001 -> 0.0978679932242825
- link link2: mass 0.0001 -> 0.289571136953082
- link link3: mass 0.0001 -> 0.290583243387798
- link link4: mass 0.0001 -> 0.127087348341362
- link link5: mass 0.0001 -> 0.144711242639456

File: src/piper_description/urdf/piper_no_gripper_description.xacro (robot description, xacro)
@@ -17,5 +17,5 @@
         rpy="0 0 0" />
       <mass
-        value="0.0001" />
+        value="0.162352169522719" />
       <inertia
         ixx="0.000226592553127906"
@@ -29,5 +29,5 @@
       <origin
         xyz="0 0 0"
-        rpy="1.5708 0 -1.5708" />
+        rpy="0 0 0" />
       <geometry>
         <mesh
@@ -57,5 +57,5 @@
         rpy="0 0 0" />
       <mass
-        value="0.0001" />
+        value="0.0978679932242825" />
       <inertia
         ixx="7.76684558296782E-05"
@@ -69,5 +69,5 @@
       <origin
         xyz="0 0 0"
-        rpy="1.5708 0 0" />
+        rpy="0 0 0" />
       <geometry>
         <mesh
@@ -115,5 +115,5 @@
         rpy="0 0 0" />
       <mass
-        value="0.0001" />
+        value="0.289571136953082" />
       <inertia
         ixx="0.000150112628108228"
@@ -127,5 +127,5 @@
       <origin
         xyz="0 0 0"
-        rpy="0 1.5708 -0.0873" />
+        rpy="0 0 0" />
       <geometry>
         <mesh
@@ -173,5 +173,5 @@
         rpy="0 0 0" />
       <mass
-        value="0.0001" />
+        value="0.290583243387798" />
       <inertia
         ixx="0.00022168634302318"
@@ -185,5 +185,5 @@
       <origin
         xyz="0 0 0"
-        rpy="1.4835 1.5708 0" />
+        rpy="0 0 0" />
       <geometry>
         <mesh
@@ -231,5 +231,5 @@
         rpy="0 0 0" />
       <mass
-        value="0.0001" />
+        value="0.127087348341362" />
       <inertia
         ixx="3.82011730423392E-05"
@@ -243,5 +243,5 @@
       <origin
         xyz="0 0 0"
-        rpy="1.48 0 1.5708" />
+        rpy="0 0 0" />
       <geometry>
         <mesh
@@ -289,5 +289,5 @@
         rpy="0 0 0" />
       <mass
-        value="0.0001" />
+        value="0.144711242639456" />
       <inertia
         ixx="4.39644313661978E-05"
@@ -301,5 +301,5 @@
       <origin
         xyz="0 0 0"
-        rpy="1.4835 1.5708 0" />
+        rpy="0 0 0" />
       <geometry>
         <mesh
@@ -365,5 +365,5 @@
     </plugin>
   </gazebo>
-  <gazebo reference="base_link">
+  <!-- <gazebo reference="base_link">
     <material>Gazebo/Black</material>
   </gazebo>
@@ -382,4 +382,4 @@
   <gazebo reference="link5">
     <material>Gazebo/White</material>
-  </gazebo>
+  </gazebo> -->
 </robot>

File: src/piper_description/urdf/piper_no_gripper_description_v00.urdf (robot description, URDF)
Before this commit: robot piper_description, 6 links, 5 joints
Links:
- link base_link: mass 0.0001 -> 0.162352169522719
- link link1: mass 0.0001 -> 0.0978679932242825
- link link2: mass 0.0001 -> 0.289571136953082
- link link3: mass 0.0001 -> 0.290583243387798
- link link4: mass 0.0001 -> 0.127087348341362
- link link5: mass 0.0001 -> 0.144711242639456

File: src/piper_description/urdf/piper_no_gripper_description_v00.xacro (robot description, xacro)
@@ -17,5 +17,5 @@
         rpy="0 0 0" />
       <mass
-        value="0.0001" />
+        value="0.162352169522719" />
       <inertia
         ixx="0.000226592553127906"
@@ -29,5 +29,5 @@
       <origin
         xyz="0 0 0"
-        rpy="1.5708 0 -1.5708" />
+        rpy="0 0 0" />
       <geometry>
         <mesh
@@ -57,5 +57,5 @@
         rpy="0 0 0" />
       <mass
-        value="0.0001" />
+        value="0.0978679932242825" />
       <inertia
         ixx="7.76684558296782E-05"
@@ -69,5 +69,5 @@
       <origin
         xyz="0 0 0"
-        rpy="1.5708 0 0" />
+        rpy="0 0 0" />
       <geometry>
         <mesh
@@ -115,5 +115,5 @@
         rpy="0 0 0" />
       <mass
-        value="0.0001" />
+        value="0.289571136953082" />
       <inertia
         ixx="0.000150112628108228"
@@ -127,5 +127,5 @@
       <origin
         xyz="0 0 0"
-        rpy="0 1.5708 -0.0873" />
+        rpy="0 0 0" />
       <geometry>
         <mesh
@@ -176,5 +176,5 @@
         rpy="0 0 0" />
       <mass
-        value="0.0001" />
+        value="0.290583243387798" />
       <inertia
         ixx="0.00022168634302318"
@@ -188,5 +188,5 @@
       <origin
         xyz="0 0 0"
-        rpy="1.4835 1.5708 0" />
+        rpy="0 0 0" />
       <geometry>
         <mesh
@@ -237,5 +237,5 @@
         rpy="0 0 0" />
       <mass
-        value="0.0001" />
+        value="0.127087348341362" />
       <inertia
         ixx="3.82011730423392E-05"
@@ -249,5 +249,5 @@
       <origin
         xyz="0 0 0"
-        rpy="1.48 0 1.5708" />
+        rpy="0 0 0" />
       <geometry>
         <mesh
@@ -295,5 +295,5 @@
         rpy="0 0 0" />
       <mass
-        value="0.0001" />
+        value="0.144711242639456" />
       <inertia
         ixx="4.39644313661978E-05"
@@ -307,5 +307,5 @@
       <origin
         xyz="0 0 0"
-        rpy="1.4835 1.5708 0" />
+        rpy="0 0 0" />
       <geometry>
         <mesh
@@ -371,5 +371,5 @@
     </plugin>
   </gazebo>
-  <gazebo reference="base_link">
+  <!-- <gazebo reference="base_link">
     <material>Gazebo/Black</material>
   </gazebo>
@@ -388,4 +388,4 @@
   <gazebo reference="link5">
     <material>Gazebo/White</material>
-  </gazebo>
+  </gazebo> -->
 </robot>
