Commit message: 修改urdf为正确坐标系

File: src/piper_description/urdf/piper_no_gripper_description.xacro (robot description, xacro)
@@ -14,15 +14,15 @@
     <inertial>
       <origin
-        xyz="-0.00973928490005031 1.83127089286717E-06 0.0410140167677137"
-        rpy="0 0 0" />
-      <mass
-        value="0.162352169522719" />
-      <inertia
-        ixx="0.000226592553127906"
-        ixy="-7.33974356968615E-08"
-        ixz="2.13221970218122E-06"
-        iyy="0.000269447877479622"
-        iyz="8.15167478682596E-09"
-        izz="0.000222318286704" />
+        xyz="-0.00979274765955341 1.82905827587138E-06 0.0410100126360189"
+        rpy="0 0 0" />
+      <mass
+        value="0.162548567403693" />
+      <inertia
+        ixx="0.000226596924525071"
+        ixy="-7.33972270153965E-08"
+        ixz="2.13249977802622E-06"
+        iyy="0.000269444772561524"
+        iyz="8.15169009611054E-09"
+        izz="0.000222318258878636" />
     </inertial>
     <visual>
@@ -54,5 +54,5 @@
     <inertial>
       <origin
-        xyz="0.00131676031927021 0.000310288842008365 -0.00922874512303438"
+        xyz="0.00131676031927024 0.000310288842008612 -0.00922874512303437"
         rpy="0 0 0" />
       <mass
@@ -60,9 +60,9 @@
       <inertia
         ixx="7.76684558296782E-05"
-        ixy="1.09084650459916E-07"
-        ixz="-1.97480532432411E-06"
-        iyy="9.24967780161546E-05"
-        iyz="9.91284646834672E-07"
-        izz="8.24589062407806E-05" />
+        ixy="1.09084650459924E-07"
+        ixz="-1.9748053243241E-06"
+        iyy="9.24967780161547E-05"
+        iyz="9.91284646834582E-07"
+        izz="8.24589062407807E-05" />
     </inertial>
     <visual>
@@ -112,15 +112,15 @@
     <inertial>
       <origin
-        xyz="0.147615838821413 -0.0174259998251394 0.00175952516190707"
-        rpy="0 0 0" />
-      <mass
-        value="0.289571136953082" />
-      <inertia
-        ixx="0.000150112628108228"
-        ixy="8.58974959950769E-05"
-        ixz="-1.07428153464284E-06"
-        iyy="0.00172585302855383"
-        iyz="-9.93704792239676E-07"
-        izz="0.00177445942914759" />
+        xyz="0.148793602378802 -0.00242026983944119 0.00175154638467948"
+        rpy="0 0 0" />
+      <mass
+        value="0.290888938633388" />
+      <inertia
+        ixx="0.000148959640166183"
+        ixy="-7.37750384371657E-05"
+        ixz="-9.68688405196236E-07"
+        iyy="0.00172800946632652"
+        iyz="-1.09692225564224E-06"
+        izz="0.0017754628344594" />
     </inertial>
     <visual>
@@ -153,5 +153,5 @@
     <origin
       xyz="0 0 0"
-      rpy="1.5708 -0.10095 -1.5708" />
+      rpy="1.5708 0 -1.5708" />
     <parent
       link="link1" />
@@ -170,15 +170,15 @@
     <inertial>
       <origin
-        xyz="0.0156727239770991 0.104466514402189 0.000508486576356504"
-        rpy="0 0 0" />
-      <mass
-        value="0.290583243387798" />
-      <inertia
-        ixx="0.00022168634302318"
-        ixy="-7.57426147001315E-06"
-        ixz="-6.36999759250492E-07"
-        iyy="0.000100859159512329"
-        iyz="-8.16199264787698E-07"
-        izz="0.000241839306422341" />
+        xyz="-0.0996835215213704 0.0349477226691318 0.000508025815507312"
+        rpy="0 0 0" />
+      <mass
+        value="0.290847697793211" />
+      <inertia
+        ixx="0.000107879011637167"
+        ixy="2.92669521203626E-05"
+        ixz="6.825922326238E-07"
+        iyy="0.000214751671792086"
+        iyz="-7.78469047878196E-07"
+        izz="0.000241923439340319" />
     </inertial>
     <visual>
@@ -210,6 +210,6 @@
     type="revolute">
     <origin
-      xyz="0.28503 0 0"
-      rpy="0 0 1.3826" />
+      xyz="0.28358 0.028726 0"
+      rpy="0 0 0.10095" />
     <parent
       link="link2" />
@@ -228,15 +228,15 @@
     <inertial>
       <origin
-        xyz="0.000276464622388145 -0.00102803669324856 -0.00472830700561582"
+        xyz="0.000276464622387979 -0.00102803669324875 -0.00472830700561663"
         rpy="0 0 0" />
       <mass
         value="0.127087348341362" />
       <inertia
-        ixx="3.82011730423392E-05"
-        ixy="-4.92358350916331E-08"
-        ixz="4.89589432971791E-08"
-        iyy="4.87048555222583E-05"
-        iyz="6.70802942501353E-08"
-        izz="4.10592077565539E-05" />
+        ixx="3.82011730423416E-05"
+        ixy="-4.92358350897513E-08"
+        ixz="4.89589432973119E-08"
+        iyy="4.87048555222578E-05"
+        iyz="6.70802942500512E-08"
+        izz="4.10592077565559E-05" />
     </inertial>
     <visual>
@@ -268,6 +268,6 @@
     type="revolute">
     <origin
-      xyz="0.021984 0.25075 0"
-      rpy="-1.5708 0 0" />
+      xyz="-0.24221 0.068514 0"
+      rpy="-1.5708 0 1.3826" />
     <parent
       link="link3" />
@@ -286,15 +286,15 @@
     <inertial>
       <origin
-        xyz="8.82262433637704E-05 0.0566829014808264 -0.00196119720482555"
-        rpy="0 0 0" />
-      <mass
-        value="0.144711242639456" />
-      <inertia
-        ixx="4.39644313661978E-05"
-        ixy="-3.59259686449865E-08"
-        ixz="-1.89747741592145E-08"
-        iyy="5.6317392095077E-05"
-        iyz="-2.1540716689678E-07"
-        izz="4.88713664675246E-05" />
+        xyz="8.82262433516967E-05 0.0566829014808256 -0.00196119720482461"
+        rpy="0 0 0" />
+      <mass
+        value="0.144711242639457" />
+      <inertia
+        ixx="4.39644313662493E-05"
+        ixy="-3.59259686444846E-08"
+        ixz="-1.89747741386183E-08"
+        iyy="5.63173920951307E-05"
+        iyz="-2.1540716689785E-07"
+        izz="4.88713664675268E-05" />
     </inertial>
     <visual>

File: src/piper_description/urdf/piper_no_gripper_description_v00.urdf (robot description, URDF)
Before this commit: robot piper_description, 6 links, 5 joints
Links:
- link base_link: mass 0.162352169522719 -> 0.162548567403693
- link link2: mass 0.289571136953082 -> 0.290888938633388
- link link3: mass 0.290583243387798 -> 0.290847697793211
- link link5: mass 0.144711242639456 -> 0.144711242639457
Joints:
- joint joint2: origin xyz=0 0 0 rpy=1.5708 -0.135857 -1.5708 -> xyz=0 0 0 rpy=1.5708 -0.034907 -1.5708
- joint joint3: origin xyz=0.28503 0 0 rpy=0 0 1.347693 -> xyz=0.28358 0.028726 0 rpy=0 0 0.06604341
- joint joint4: origin xyz=0.021984 0.25075 0 rpy=-1.5708 0 0 -> xyz=-0.24221 0.068514 0 rpy=-1.5708 0 1.3826

File: src/piper_description/urdf/piper_no_gripper_description_v00.xacro (robot description, xacro)
@@ -14,15 +14,15 @@
     <inertial>
       <origin
-        xyz="-0.00973928490005031 1.83127089286717E-06 0.0410140167677137"
-        rpy="0 0 0" />
-      <mass
-        value="0.162352169522719" />
-      <inertia
-        ixx="0.000226592553127906"
-        ixy="-7.33974356968615E-08"
-        ixz="2.13221970218122E-06"
-        iyy="0.000269447877479622"
-        iyz="8.15167478682596E-09"
-        izz="0.000222318286704" />
+        xyz="-0.00979274765955341 1.82905827587138E-06 0.0410100126360189"
+        rpy="0 0 0" />
+      <mass
+        value="0.162548567403693" />
+      <inertia
+        ixx="0.000226596924525071"
+        ixy="-7.33972270153965E-08"
+        ixz="2.13249977802622E-06"
+        iyy="0.000269444772561524"
+        iyz="8.15169009611054E-09"
+        izz="0.000222318258878636" />
     </inertial>
     <visual>
@@ -54,5 +54,5 @@
     <inertial>
       <origin
-        xyz="0.00131676031927021 0.000310288842008365 -0.00922874512303438"
+        xyz="0.00131676031927024 0.000310288842008612 -0.00922874512303437"
         rpy="0 0 0" />
       <mass
@@ -60,9 +60,9 @@
       <inertia
         ixx="7.76684558296782E-05"
-        ixy="1.09084650459916E-07"
-        ixz="-1.97480532432411E-06"
-        iyy="9.24967780161546E-05"
-        iyz="9.91284646834672E-07"
-        izz="8.24589062407806E-05" />
+        ixy="1.09084650459924E-07"
+        ixz="-1.9748053243241E-06"
+        iyy="9.24967780161547E-05"
+        iyz="9.91284646834582E-07"
+        izz="8.24589062407807E-05" />
     </inertial>
     <visual>
@@ -112,15 +112,15 @@
     <inertial>
       <origin
-        xyz="0.147615838821413 -0.0174259998251394 0.00175952516190707"
-        rpy="0 0 0" />
-      <mass
-        value="0.289571136953082" />
-      <inertia
-        ixx="0.000150112628108228"
-        ixy="8.58974959950769E-05"
-        ixz="-1.07428153464284E-06"
-        iyy="0.00172585302855383"
-        iyz="-9.93704792239676E-07"
-        izz="0.00177445942914759" />
+        xyz="0.148793602378802 -0.00242026983944119 0.00175154638467948"
+        rpy="0 0 0" />
+      <mass
+        value="0.290888938633388" />
+      <inertia
+        ixx="0.000148959640166183"
+        ixy="-7.37750384371657E-05"
+        ixz="-9.68688405196236E-07"
+        iyy="0.00172800946632652"
+        iyz="-1.09692225564224E-06"
+        izz="0.0017754628344594" />
     </inertial>
     <visual>
@@ -151,10 +151,7 @@
     name="joint2"
     type="revolute">
-    <!-- <origin
+    <origin
       xyz="0 0 0"
-      rpy="1.5708 -0.10095 -1.5708" /> -->
-    <origin
-      xyz="0 0 0"
-      rpy="1.5708 -0.135857 -1.5708" />
+      rpy="1.5708 -0.034907 -1.5708" />
     <parent
       link="link1" />
@@ -173,15 +170,15 @@
     <inertial>
       <origin
-        xyz="0.0156727239770991 0.104466514402189 0.000508486576356504"
-        rpy="0 0 0" />
-      <mass
-        value="0.290583243387798" />
-      <inertia
-        ixx="0.00022168634302318"
-        ixy="-7.57426147001315E-06"
-        ixz="-6.36999759250492E-07"
-        iyy="0.000100859159512329"
-        iyz="-8.16199264787698E-07"
-        izz="0.000241839306422341" />
+        xyz="-0.0996835215213704 0.0349477226691318 0.000508025815507312"
+        rpy="0 0 0" />
+      <mass
+        value="0.290847697793211" />
+      <inertia
+        ixx="0.000107879011637167"
+        ixy="2.92669521203626E-05"
+        ixz="6.825922326238E-07"
+        iyy="0.000214751671792086"
+        iyz="-7.78469047878196E-07"
+        izz="0.000241923439340319" />
     </inertial>
     <visual>
@@ -212,10 +209,7 @@
     name="joint3"
     type="revolute">
-    <!-- <origin
-      xyz="0.28503 0 0"
-      rpy="0 0 1.3826" /> -->
-    <origin
-      xyz="0.28503 0 0"
-      rpy="0 0 1.347693" />
+    <origin
+      xyz="0.28358 0.028726 0"
+      rpy="0 0 0.06604341" />
     <parent
       link="link2" />
@@ -234,15 +228,15 @@
     <inertial>
       <origin
-        xyz="0.000276464622388145 -0.00102803669324856 -0.00472830700561582"
+        xyz="0.000276464622387979 -0.00102803669324875 -0.00472830700561663"
         rpy="0 0 0" />
       <mass
         value="0.127087348341362" />
       <inertia
-        ixx="3.82011730423392E-05"
-        ixy="-4.92358350916331E-08"
-        ixz="4.89589432971791E-08"
-        iyy="4.87048555222583E-05"
-        iyz="6.70802942501353E-08"
-        izz="4.10592077565539E-05" />
+        ixx="3.82011730423416E-05"
+        ixy="-4.92358350897513E-08"
+        ixz="4.89589432973119E-08"
+        iyy="4.87048555222578E-05"
+        iyz="6.70802942500512E-08"
+        izz="4.10592077565559E-05" />
     </inertial>
     <visual>
@@ -274,6 +268,6 @@
     type="revolute">
     <origin
-      xyz="0.021984 0.25075 0"
-      rpy="-1.5708 0 0" />
+      xyz="-0.24221 0.068514 0"
+      rpy="-1.5708 0 1.3826" />
     <parent
       link="link3" />
@@ -292,15 +286,15 @@
     <inertial>
       <origin
-        xyz="8.82262433637704E-05 0.0566829014808264 -0.00196119720482555"
-        rpy="0 0 0" />
-      <mass
-        value="0.144711242639456" />
-      <inertia
-        ixx="4.39644313661978E-05"
-        ixy="-3.59259686449865E-08"
-        ixz="-1.89747741592145E-08"
-        iyy="5.6317392095077E-05"
-        iyz="-2.1540716689678E-07"
-        izz="4.88713664675246E-05" />
+        xyz="8.82262433516967E-05 0.0566829014808256 -0.00196119720482461"
+        rpy="0 0 0" />
+      <mass
+        value="0.144711242639457" />
+      <inertia
+        ixx="4.39644313662493E-05"
+        ixy="-3.59259686444846E-08"
+        ixz="-1.89747741386183E-08"
+        iyy="5.63173920951307E-05"
+        iyz="-2.1540716689785E-07"
+        izz="4.88713664675268E-05" />
     </inertial>
     <visual>
